Commit message: 完成基于ros2_control的阿克曼模型创建

File: src/agents_cpp/urdf/robot.urdf.xacro (robot description, xacro)
@@ -1,4 +1,4 @@
 <?xml version="1.0"?>
-<robot name="integrator" xmlns:xacro="http://www.ros.org/wiki/xacro">
+<robot name="bicyble" xmlns:xacro="http://www.ros.org/wiki/xacro">
   <!-- 定义带命名空间的参数 -->
   <xacro:arg name="robot_namespace" default="" />
@@ -12,7 +12,6 @@
       <origin xyz="0 0 0" rpy="0 0 0"/>
       <geometry>
-        <mesh filename="package://agents_py/meshes/ardrone.dae" scale="1.0 1.0 1.0"/>
-        <!-- <mesh filename="package://odom_differential/meshes/747-400/747-400.dae" scale="0.1 0.1 0.1"/> -->
-        <!-- <mesh filename="package://odom_differential/meshes/glider/glider.dae" scale="0.1 0.1 0.1"/> -->
+        <box size="0.5 0.5 0.3"/>
+        <!-- <mesh filename="package://agents_cpp/meshes/xxx" scale="0.1 0.1 0.1"/> -->
       </geometry>
     </visual>
