Commit message: ..

File: src/agents_cpp/urdf/car.gz_ros2_control.urdf.xacro (robot description, xacro)
@@ -3,19 +3,24 @@
     <xacro:arg name="robot_namespace" default="" />
     <xacro:property name="ns" value="$(arg robot_namespace)" />
-    <xacro:include filename="$(find agents_cpp)/urdf/car.urdf.xacro" />
+    <xacro:arg name="joint_prefix" default=""/>
+    <xacro:property name="jp" value="$(arg joint_prefix)" />
+    <!-- 新增：控制器配置文件路径作为参数 -->
+    <xacro:arg name="controllers_yaml" default="" />
+    <xacro:property name="cy" value="$(arg controllers_yaml)" />
+    <xacro:include filename="$(find agents_cpp)/urdf/car.xacro" />
     <!-- ros2_control 硬件接口（使用 mock 组件做演示） -->
-    <ros2_control name="${ns}car" type="system">
+    <ros2_control name="${jp}car" type="system">
         <hardware>
-            <param name="calculate_dynamics">true</param>
+            <!-- <param name="calculate_dynamics">true</param> -->
             <!-- <plugin>mock_components/GenericSystem</plugin> -->
             <plugin>gz_ros2_control/GazeboSimSystem</plugin>
         </hardware>
         <!-- 后轮：速度控制接口（diff_drive） -->
-        <joint name="${ns}rear_left_wheel_joint">
+        <joint name="${jp}rear_left_wheel_joint">
             <command_interface name="velocity" />
             <state_interface name="position" />
             <state_interface name="velocity" />
         </joint>
-        <joint name="${ns}rear_right_wheel_joint">
+        <joint name="${jp}rear_right_wheel_joint">
             <command_interface name="velocity" />
             <state_interface name="position" />
@@ -23,10 +28,10 @@
         </joint>
         <!-- 前轮转向：位置控制接口（给定转向角） -->
-        <joint name="${ns}front_left_steer_joint">
+        <joint name="${jp}front_left_steer_joint">
             <command_interface name="position" />
             <state_interface name="position" />
             <state_interface name="velocity" />
         </joint>
-        <joint name="${ns}front_right_steer_joint">
+        <joint name="${jp}front_right_steer_joint">
             <command_interface name="position" />
             <state_interface name="position" />
@@ -34,9 +39,9 @@
         </joint>
         <!-- 前轮滚动：仅状态 -->
-        <joint name="${ns}front_left_wheel_joint">
+        <joint name="${jp}front_left_wheel_joint">
             <state_interface name="position" />
             <state_interface name="velocity" />
         </joint>
-        <joint name="${ns}front_right_wheel_joint">
+        <joint name="${jp}front_right_wheel_joint">
             <state_interface name="position" />
             <state_interface name="velocity" />
@@ -44,6 +49,13 @@
     </ros2_control>
     <gazebo>
+        <!-- <plugin filename="gz_ros2_control-system" name="gz_ros2_control::GazeboSimROS2ControlPlugin"> -->
         <plugin filename="gz_ros2_control-system" name="gz_ros2_control::GazeboSimROS2ControlPlugin">
-            <parameters>$(find agents_cpp)/config/controllers.yaml</parameters>
+            <ros>
+                <namespace>${ns}</namespace>
+                <remapping>ackermann_steering_controller/tf_odometry:=/tf</remapping>
+            </ros>
+            <!-- <parameters>$(find agents_cpp)/config/controllers.yaml</parameters> -->
+            <!-- <parameters>$(find agents_cpp)/config/agent0_controllers.yaml</parameters> -->
+            <parameters>${cy}</parameters>
         </plugin>
     </gazebo>

File: src/agents_cpp/urdf/car.ros2_control.xacro (robot description, xacro)
@@ -3,6 +3,8 @@
     <xacro:arg name="robot_namespace" default="" />
     <xacro:property name="ns" value="$(arg robot_namespace)" />
+    <xacro:arg name="joint_prefix" default="" />
+    <xacro:property name="jp" value="$(arg joint_prefix)" />
     <!-- ros2_control 硬件接口（使用 mock 组件做演示） -->
-    <ros2_control name="${ns}car" type="system">
+    <ros2_control name="${jp}car" type="system">
         <hardware>
             <param name="calculate_dynamics">true</param>
@@ -14,10 +16,10 @@
         </hardware>
         <!-- 后轮：速度控制接口（diff_drive） -->
-        <joint name="${ns}rear_left_wheel_joint">
+        <joint name="${jp}rear_left_wheel_joint">
             <command_interface name="velocity" />
             <state_interface name="position" />
             <state_interface name="velocity" />
         </joint>
-        <joint name="${ns}rear_right_wheel_joint">
+        <joint name="${jp}rear_right_wheel_joint">
             <command_interface name="velocity" />
             <state_interface name="position" />
@@ -25,10 +27,10 @@
         </joint>
         <!-- 前轮转向：位置控制接口（给定转向角） -->
-        <joint name="${ns}front_left_steer_joint">
+        <joint name="${jp}front_left_steer_joint">
             <command_interface name="position" />
             <state_interface name="position" />
             <state_interface name="velocity" />
         </joint>
-        <joint name="${ns}front_right_steer_joint">
+        <joint name="${jp}front_right_steer_joint">
             <command_interface name="position" />
             <state_interface name="position" />
@@ -36,9 +38,9 @@
         </joint>
         <!-- 前轮滚动：仅状态 -->
-        <joint name="${ns}front_left_wheel_joint">
+        <joint name="${jp}front_left_wheel_joint">
             <state_interface name="position" />
             <state_interface name="velocity" />
         </joint>
-        <joint name="${ns}front_right_wheel_joint">
+        <joint name="${jp}front_right_wheel_joint">
             <state_interface name="position" />
             <state_interface name="velocity" />

File: src/agents_cpp/urdf/car.urdf.xacro (robot description, xacro)
@@ -4,114 +4,8 @@
     <xacro:arg name="robot_namespace" default="" />
     <xacro:property name="ns" value="$(arg robot_namespace)" />
+    <xacro:arg name="joint_prefix" default=""/>
+    <xacro:property name="jp" value="$(arg joint_prefix)" />
     <!-- 引入子文件 -->
-    <xacro:include filename="$(find agents_cpp)/urdf/wheel.xacro" />
-    <xacro:include filename="$(find agents_cpp)/urdf/steering_wheel.xacro" />
-    <!-- 通用参数 -->
-    <xacro:property name="body_height" value="0.3" />
-    <xacro:property name="body_width" value="0.5" />
-    <xacro:property name="wheel_radius" value="0.1" />
-    <xacro:property name="wheel_width" value="0.05" />
-    <xacro:property name="wheelbase" value="0.6" />
-    <xacro:property name="track" value="0.4" />
-    <!-- odom -->
-    <link name="${ns}odom" />
-    <!-- 车体底座 -->
-    <link name="${ns}base_footprint">
-        <!-- base_footprint 一般是一个虚拟参考平面，不参与碰撞 -->
-        <visual>
-            <origin xyz="0 0 0" rpy="0 0 0" />
-            <geometry>
-                <sphere radius="0.01" />
-            </geometry>
-            <material name="transparent">
-                <color rgba="0 0 0 0" />
-            </material>
-        </visual>
-        <inertial>
-            <!-- 虚拟质量极小，仅用于计算结构完整性 -->
-            <mass value="0.01" />
-            <origin xyz="0 0 0" rpy="0 0 0" />
-            <inertia ixx="1e-6" ixy="0" ixz="0" iyy="1e-6" iyz="0" izz="1e-6" />
-        </inertial>
-    </link>
-    <!-- base_footprint -> base_link 固定连接 -->
-    <joint name="${ns}base_footprint_joint" type="fixed">
-        <parent link="${ns}base_footprint" />
-        <child link="${ns}base_link" />
-        <origin xyz="0 0 $(eval ${body_height} - ${wheel_radius})" rpy="0 0 0" />
-    </joint>
-    <!-- 车体 -->
-    <link name="${ns}base_link">
-        <visual>
-            <origin xyz="0 0 0" rpy="0 0 0" />
-            <geometry>
-                <box size="${body_width} ${body_width} ${body_height}" />
-            </geometry>
-            <material name="yellow">
-                <color rgba="1.0 1.0 0.0 1" />
-            </material>
-        </visual>
-        <collision>
-            <geometry>
-                <box size="${body_width} ${body_width} ${body_height}" />
-            </geometry>
-        </collision>
-        <inertial>
-            <!-- 车体质量与惯量，可按几何估算 -->
-            <mass value="5.0" />
-            <origin xyz="0 0 0" rpy="0 0 0" />
-            <inertia
-                ixx="0.10"
-                ixy="0.0"
-                ixz="0.0"
-                iyy="0.20"
-                iyz="0.0"
-                izz="0.20" />
-        </inertial>
-    </link>
-    <!-- odom -> base_footprint 固定连接 -->
-    <joint name="${ns}odom_joint" type="fixed">
-        <parent link="${ns}odom" />
-        <child link="${ns}base_footprint" />
-        <origin xyz="0 0 0" rpy="0 0 0" />
-    </joint>
-    <!-- =================== -->
-    <!--     后轮：复用wheel  -->
-    <!-- =================== -->
-    <!-- 后左轮：车体后方(-wheelbase/2)，左(+track/2) -->
-    <xacro:wheel
-        parent="${ns}base_link"
-        name="${ns}rear_left_wheel"
-        xyz="$(eval -${wheelbase} / 2) $(eval ${track} / 2) $(eval -${wheel_radius})"
-        radius="${wheel_radius}"
-        width="${wheel_width}"
-        axis="0 1 0" />
-    <!-- 后右轮 -->
-    <xacro:wheel
-        parent="${ns}base_link"
-        name="${ns}rear_right_wheel"
-        xyz="$(eval -${wheelbase} / 2) $(eval -${track} / 2) $(eval -${wheel_radius})"
-        radius="${wheel_radius}"
-        width="${wheel_width}"
-        axis="0 1 0" />
-    <!-- =================== -->
-    <!--   前轮：复用steering -->
-    <!-- =================== -->
-    <!-- 前左转向轮 -->
-    <xacro:steering_wheel
-        parent="${ns}base_link"
-        name_prefix="${ns}front_left"
-        xyz="$(eval  ${wheelbase} / 2) $(eval ${track} / 2) 0"
-        steer_limit="0.7"
-        radius="${wheel_radius}"
-        width="${wheel_width}" />
-    <!-- 前右转向轮 -->
-    <xacro:steering_wheel
-        parent="${ns}base_link"
-        name_prefix="${ns}front_right"
-        xyz="$(eval  ${wheelbase} / 2) $(eval -${track} / 2) 0"
-        steer_limit="0.7"
-        radius="${wheel_radius}"
-        width="${wheel_width}" />
+    <xacro:include filename="$(find agents_cpp)/urdf/car.xacro" />
     <xacro:include filename="$(find agents_cpp)/urdf/car.ros2_control.xacro" />
 </robot>

File: src/agents_cpp/urdf/steering_wheel.xacro (robot description, xacro)
@@ -29,4 +29,18 @@
         </material>
       </visual>
+      <!-- collision：与 visual 一致 -->
+      <collision>
+        <geometry>
+          <box size="0.05 0.05 0.05"/>
+        </geometry>
+      </collision>
+      <!-- inertial：质量、惯性矩，基于 0.05m 立方体 -->
+      <inertial>
+        <mass value="0.1"/>
+        <origin xyz="0 0 0" rpy="0 0 0"/>
+        <!-- 惯性矩基于实心立方体 I = (1/6) m * a^2 -->
+        <!-- a = 0.05m,  m=0.1kg → I = 0.1 * 0.05^2 / 6 = 4.1667e-05 -->
+        <inertia ixx="4.17e-05" iyy="4.17e-05" izz="4.17e-05" ixy="0.0" ixz="0.0" iyz="0.0"/>
+      </inertial>
     </link>
     <!-- 车身 -> 转向支架：绕Z轴转向 -->
